Commit message: updated stl and urdf file to reflect the new dimensions

File: autorally_description/urdf/autoRallyPlatform.urdf1.xacro (robot description, xacro)
@@ -322,5 +322,5 @@
               rpy="0 0 0"/>
       <geometry>
-        <mesh filename="package://autorally_description/urdf/autoRallyPlatformChassis.stl" scale="0.01 0.01 0.01" />
+        <mesh filename="package://autorally_description/urdf/autoRallyChassis.stl" scale="0.01 0.01 0.01" />
       </geometry>
       <material name="chassis_mat"/>
@@ -330,5 +330,5 @@
               rpy="0 0 0"/>
       <geometry>
-        <mesh filename="package://autorally_description/urdf/autoRallyPlatformChassis.stl" scale="1.01 1.01 1.01" />
+        <mesh filename="package://autorally_description/urdf/autoRallyChassis.stl" scale="1.01 1.01 1.01" />
       </geometry>
     </collision>
