Commit message: simplified wheel models so simulation is faster and updated all related files

File: autorally_description/urdf/autoRallyPlatform.urdf.xacro (robot description, xacro)
@@ -190,5 +190,5 @@
       <limit effort="${axle_eff_limit}" velocity="${axle_vel_limit}"/>
       <!-- <dynamics damping="0.015" friction="0.0"/> -->
-      <dynamics damping="0.003" friction="0.5"/>
+      <dynamics damping="0.001" friction="0.5"/>
     </joint>
 <!--    <gazebo reference="${lr_prefix}_${fr_prefix}_axle">
@@ -212,5 +212,5 @@
         <origin xyz="0 0 0"/>
         <geometry>
-          <mesh filename="${wheel_model}" scale="0.01 0.01 0.01" />
+          <mesh filename="${wheel_model}" />
         </geometry>
       </visual>
@@ -218,5 +218,5 @@
         <origin xyz="0 0 0"/>
         <geometry>
-          <mesh filename="${wheel_model}" scale="0.01 0.01 0.01" />
+          <mesh filename="${wheel_model}" />
         </geometry>
       </collision>
@@ -224,5 +224,5 @@
         <origin xyz="0 0 0"/>
         <geometry>
-          <mesh filename="${wheel_model}" scale="0.01 0.01 0.01" />
+          <mesh filename="${wheel_model}" />
         </geometry>
       </collision>

Commit message: Updated steer angle of simulator

File: autorally_description/urdf/autoRallyPlatform.urdf.xacro (robot description, xacro)
@@ -24,5 +24,5 @@
   <!-- Degree-to-radian conversions -->
   <xacro:property name="degrees_45" value="0.785398163"/>
-  <xacro:property name="degrees_25" value="0.436332313"/>
+  <xacro:property name="degrees_21" value="0.3665191429"/>
   <xacro:property name="degrees_90" value="1.57079633"/>
   <!-- chassis_length is measured along the x axis, chassis_width
@@ -264,5 +264,5 @@
       <!-- cant the front wheels to improve traction -->
       <axis xyz="0 ${-lr_reflect*0.09950372}  0.99503719"/>
-      <limit lower="${-degrees_25}" upper="${degrees_25}"
+      <limit lower="${-degrees_21}" upper="${degrees_21}"
              effort="${servo_stall_torque}" velocity="${servo_no_load_speed}"/>
     </joint>

Commit message: Merge?

File: autorally_description/urdf/autoRallyPlatform.urdf.xacro (robot description, xacro)
@@ -133,5 +133,5 @@
       <limit lower="${-front_wheel_travel / 2}" upper="${front_wheel_travel / 2}"
              effort="${front_shock_eff_limit}" velocity="${shock_vel_limit}"/>
-      <dynamics damping="88" friction="0.0001"
+      <dynamics damping="100" friction="0.0001"
                 spring_stiffness="3152" spring_reference="0.08"/>
     </joint>
@@ -161,5 +161,5 @@
       <limit lower="${-rear_wheel_travel / 2}" upper="${rear_wheel_travel / 2}"
              effort="${rear_shock_eff_limit}" velocity="${shock_vel_limit}"/>
-      <dynamics damping="0" friction="0.0"/>
+      <dynamics damping="100" friction="0.0"/>
     </joint>
     <transmission name="${lr_prefix}_${fr_prefix}_shock_trans">
@@ -363,5 +363,5 @@
   </link>
   <joint name="imu_joint" type="fixed">
-    <origin xyz="0 0 0" rpy="0 0 0"/>
+    <origin xyz="0 0 0" rpy="3.14159 0 0"/>
     <parent link="base_link"/>
     <child link="imu_link"/>
@@ -554,5 +554,5 @@
       <frameId>imu_link</frameId>
       <topicName>imu</topicName>
-      <rpyOffset>0 0 0</rpyOffset>
+      <rpyOffset>3.14159 0 0</rpyOffset>
       <xyzOffset>0 0 0</xyzOffset>
       <gaussianNoise>0.00000001</gaussianNoise>

Commit message: Removed IMU roll i was playing with

File: autorally_description/urdf/autoRallyPlatform.urdf.xacro (robot description, xacro)
@@ -363,5 +363,5 @@
   </link>
   <joint name="imu_joint" type="fixed">
-    <origin xyz="0 0 0" rpy="3.14159 0 0"/>
+    <origin xyz="0 0 0" rpy="0 0 0"/>
     <parent link="base_link"/>
     <child link="imu_link"/>
@@ -554,5 +554,5 @@
       <frameId>imu_link</frameId>
       <topicName>imu</topicName>
-      <rpyOffset>3.14159 0 0</rpyOffset>
+      <rpyOffset>0 0 0</rpyOffset>
       <xyzOffset>0 0 0</xyzOffset>
       <gaussianNoise>0.00000001</gaussianNoise>

Commit message: Added back in damping for rear shocks that was removed at some point

File: autorally_description/urdf/autoRallyPlatform.urdf.xacro (robot description, xacro)
@@ -161,5 +161,5 @@
       <limit lower="${-rear_wheel_travel / 2}" upper="${rear_wheel_travel / 2}"
              effort="${rear_shock_eff_limit}" velocity="${shock_vel_limit}"/>
-      <dynamics damping="0" friction="0.0"/>
+      <dynamics damping="88" friction="0.0"/>
     </joint>
     <transmission name="${lr_prefix}_${fr_prefix}_shock_trans">

Commit message: Added Vehicle Textures

File: autorally_description/urdf/autoRallyPlatform.urdf.xacro (robot description, xacro)
@@ -319,7 +319,6 @@
               rpy="0 0 0"/>
       <geometry>
-        <mesh filename="package://autorally_description/urdf/autoRallyPlatform.stl" scale="0.01 0.01 0.01" />
-      </geometry>
-      <material name="chassis_mat"/>
+        <mesh filename="package://autorally_description/urdf/Vehicle_Texture.dae" scale="1 1 1" />
+      </geometry>
     </visual>
     <collision>
@@ -327,5 +326,5 @@
               rpy="0 0 0"/>
       <geometry>
-        <mesh filename="package://autorally_description/urdf/autoRallyPlatform.stl" scale="0.01 0.01 0.01" />
+        <mesh filename="package://autorally_description/urdf/Vehicle_Texture.dae" scale="1 1 1" />
       </geometry>
     </collision>
@@ -340,5 +339,4 @@
   </link>
   <gazebo reference="chassis">
-    <material>Gazebo/Grey</material>
     <mu1>0.2</mu1>
     <mu2>0.2</mu2>

Commit message: made final changes

File: autorally_description/urdf/autoRallyPlatform.urdf.xacro (robot description, xacro)
@@ -394,32 +394,4 @@
     </inertial>
   </link>
-  <joint name="side_camera_joint" type="fixed">
-    <axis xyz="0 1 0" />
-    <origin xyz="0 -3 0" rpy="0 0 1.5708"/>
-    <parent link="base_link"/>
-    <child link="side_camera_link"/>
-  </joint>
-  <!-- Camera -->
-  <link name="side_camera_link">
-    <!-- <collision>
-      <origin xyz="0 0 0" rpy="0 0 0"/>
-      <geometry>
-        <box size="0.05 0.05 0.05"/>
-      </geometry>
-    </collision>
-    <visual>
-      <origin xyz="0 0 0" rpy="0 0 0"/>
-      <geometry>
-        <box size="0.05 0.05 0.05"/>
-      </geometry>
-      <material name="red"/>
-    </visual>
-    -->
-    <inertial>
-      <mass value="1e-5" />
-      <origin xyz="0 0 0" rpy="0 0 0"/>
-      <inertia ixx="1e-6" ixy="0" ixz="0" iyy="1e-6" iyz="0" izz="1e-6" />
-    </inertial>
-  </link>
   <!-- camera -->
   <gazebo reference="camera_link">
@@ -475,44 +447,4 @@
         <distortionK3>-0.000165</distortionK3>
         <distortionT1>-0.000336</distortionT1>
-        <distortionT2>0.0</distortionT2> -->
-      </plugin>
-    </sensor>
-  </gazebo>
-   <!-- camera -->
-  <gazebo reference="side_camera_link">
-    <sensor type="camera" name="camera_side">
-      <update_rate>30.0</update_rate>
-      <camera name="side">
-        <horizontal_fov>1.3962634</horizontal_fov>
-        <image>
-          <width>1280</width>
-          <height>1024</height>
-          <format>R8G8B8</format>
-        </image>
-        <clip>
-          <near>0.02</near>
-          <far>50</far>
-        </clip>
-        <noise>
-          <type>gaussian</type>
-          <!-- Noise is sampled independently per pixel on each frame.
-               That pixel's noise value is added to each of its color
-               channels, which at that point lie in the range [0,1]. -->
-          <mean>0.0</mean>
-          <stddev>0.007</stddev>
-        </noise>
-      </camera>
-      <plugin name="camera_controller" filename="libgazebo_ros_camera.so">
-        <alwaysOn>true</alwaysOn>
-        <updateRate>0.0</updateRate>
-        <cameraName>camera_side</cameraName>
-        <imageTopicName>image_raw</imageTopicName>
-        <cameraInfoTopicName>camera_info</cameraInfoTopicName>
-        <frameName>side_camera_link</frameName>
-        <hackBaseline>0.07</hackBaseline>
-        <!-- <distortionK1>0.0</distortionK1>
-        <distortionK2>0.0</distortionK2>
-        <distortionK3>0.0</distortionK3>
-        <distortionT1>0.0</distortionT1>
         <distortionT2>0.0</distortionT2> -->
       </plugin>

Commit message: fixed urdf file

File: autorally_description/urdf/autoRallyPlatform.urdf.xacro (robot description, xacro)
@@ -347,4 +347,21 @@
     <child link="chassis"/>
   </joint>
+  <link name="gps_link">
+    <collision>
+      <geometry>
+        <box size="0.1 0.1 0.1"/>
+      </geometry>
+    </collision>
+    <inertial>
+      <mass value="1e-5" />
+      <origin xyz="0 0 0" rpy="0 0 0"/>
+      <inertia ixx="1e-6" ixy="0" ixz="0" iyy="1e-6" iyz="0" izz="1e-6" />
+    </inertial>
+  </link>
+  <joint name="gps_joint" type="fixed">
+    <origin xyz="-0.36 0 0.1359" rpy="0 0 0"/>
+    <parent link="base_link"/>
+    <child link="gps_link"/>
+  </joint>
   <link name="imu_link">
     <collision>
@@ -361,5 +378,5 @@
   </link>
   <joint name="imu_joint" type="fixed">
-    <origin xyz="0 0 0" rpy="0 0 0"/>
+    <origin xyz="-0.039 0 0.2159" rpy="0 0 0"/>
     <parent link="base_link"/>
     <child link="imu_link"/>
@@ -367,5 +384,5 @@
   <joint name="camera_joint" type="fixed">
     <axis xyz="0 0 -1" />
-    <origin xyz="0.12 0 0.05" rpy="0 0 0"/>
+    <origin xyz="0.127 0 0.2159" rpy="0 0 0"/>
     <parent link="base_link"/>
     <child link="camera_link"/>
@@ -379,6 +396,5 @@
       </geometry>
     </collision>
-<!--
-    <visual>
+    <!--<visual>
       <origin xyz="0 0 0" rpy="0 0 0"/>
       <geometry>
@@ -386,6 +402,5 @@
       </geometry>
       <material name="red"/>
-    </visual>
--->
+    </visual>-->
     <inertial>
       <mass value="1e-5" />
@@ -418,5 +433,5 @@
       <camera name="right">
         <pose>0.02 -0.07 0 0 0 0</pose>
-        <horizontal_fov>3.0</horizontal_fov>
+        <horizontal_fov>1.3962634</horizontal_fov>
         <image>
           <width>1280</width>
@@ -499,6 +514,6 @@
     <plugin name="gps" filename="libhector_gazebo_ros_gps.so">
       <updateRate>20.0</updateRate>
-      <bodyName>base_link</bodyName>
-      <frameId>base_link</frameId>
+      <bodyName>gps_link</bodyName>
+      <frameId>gps_link</frameId>
       <topicName>/gpsRoverStatus</topicName>
       <velocityTopicName>fix_velocity</velocityTopicName>

Commit message: fixed imu location to match beta

File: autorally_description/urdf/autoRallyPlatform.urdf.xacro (robot description, xacro)
@@ -378,5 +378,5 @@
   </link>
   <joint name="imu_joint" type="fixed">
-    <origin xyz="-0.039 0 0.2159" rpy="0 0 0"/>
+    <origin xyz="-0.039 0 0.0859" rpy="0 0 0"/>
     <parent link="base_link"/>
     <child link="imu_link"/>

Commit message: Added ground truth state publishing from the simulation, state estimator is no longer required in simulation

File: autorally_description/urdf/autoRallyPlatform.urdf.xacro (robot description, xacro)
@@ -141,10 +141,10 @@
       <type>transmission_interface/SimpleTransmission</type>
       <joint name="${lr_prefix}_${fr_prefix}_shock">
-        <hardwareInterface>EffortJointInterface</hardwareInterface>
+        <hardwareInterface>hardware_interface/EffortJointInterface</hardwareInterface>
       </joint>
       <actuator name="${lr_prefix}_${fr_prefix}_shock_act">
         <!-- This hardwareInterface element exists for compatibility
              with ROS Hydro. -->
-        <hardwareInterface>EffortJointInterface</hardwareInterface>
+        <hardwareInterface>hardware_interface/EffortJointInterface</hardwareInterface>
         <mechanicalReduction>1</mechanicalReduction>
       </actuator>
@@ -168,10 +168,10 @@
       <type>transmission_interface/SimpleTransmission</type>
       <joint name="${lr_prefix}_${fr_prefix}_shock">
-        <hardwareInterface>EffortJointInterface</hardwareInterface>
+        <hardwareInterface>hardware_interface/EffortJointInterface</hardwareInterface>
       </joint>
       <actuator name="${lr_prefix}_${fr_prefix}_shock_act">
         <!-- This hardwareInterface element exists for compatibility
              with ROS Hydro. -->
-        <hardwareInterface>EffortJointInterface</hardwareInterface>
+        <hardwareInterface>hardware_interface/EffortJointInterface</hardwareInterface>
         <mechanicalReduction>1</mechanicalReduction>
       </actuator>
@@ -201,10 +201,10 @@
       <type>transmission_interface/SimpleTransmission</type>
       <joint name="${lr_prefix}_${fr_prefix}_axle">
-        <hardwareInterface>EffortJointInterface</hardwareInterface>
+        <hardwareInterface>hardware_interface/EffortJointInterface</hardwareInterface>
       </joint>
       <actuator name="${lr_prefix}_${fr_prefix}_axle_act">
         <!-- This hardwareInterface element exists for compatibility
              with ROS Hydro. -->
-        <hardwareInterface>EffortJointInterface</hardwareInterface>
+        <hardwareInterface>hardware_interface/EffortJointInterface</hardwareInterface>
         <mechanicalReduction>1</mechanicalReduction>
       </actuator>
@@ -272,10 +272,10 @@
       <type>transmission_interface/SimpleTransmission</type>
       <joint name="${lr_prefix}_steering_joint">
-        <hardwareInterface>EffortJointInterface</hardwareInterface>
+        <hardwareInterface>hardware_interface/EffortJointInterface</hardwareInterface>
       </joint>
       <actuator name="${lr_prefix}_steering_act">
         <!-- This hardwareInterface element exists for compatibility
              with ROS Hydro. -->
-        <hardwareInterface>EffortJointInterface</hardwareInterface>
+        <hardwareInterface>hardware_interface/EffortJointInterface</hardwareInterface>
         <mechanicalReduction>1</mechanicalReduction>
       </actuator>
@@ -389,4 +389,42 @@
     <parent link="base_link"/>
     <child link="camera_link"/>
+  </joint>
+ <!-- <link name="odom">
+    <collision>
+      <origin xyz="0 0 0" rpy="0 0 0"/>
+      <geometry>
+        <box size="0.1 0.1 0.1"/>
+      </geometry>
+    </collision>
+    <inertial>
+      <mass value="1e-5" />
+      <origin xyz="0 0 0" rpy="0 0 0"/>
+      <inertia ixx="1e-6" ixy="0" ixz="0" iyy="1e-6" iyz="0" izz="1e-6" />
+    </inertial>
+  </link>
+  <joint name="odom_joint" type="fixed">
+    <axis xyz="0 0 0" />
+    <origin xyz="0 0 0" rpy="0 0 0"/>
+    <parent link="odom"/>
+    <child link="base_link"/>
+  </joint>
+-->
+ <link name="odom_ground_truth">
+    <collision>
+      <geometry>
+        <box size="0.1 0.1 0.1"/>
+      </geometry>
+    </collision>
+    <inertial>
+      <mass value="1e-5" />
+      <origin xyz="0 0 0" rpy="0 0 0"/>
+      <inertia ixx="1e-6" ixy="0" ixz="0" iyy="1e-6" iyz="0" izz="1e-6" />
+    </inertial>
+  </link>
+  <joint name="odom_ground_truth_joint" type="fixed">
+    <axis xyz="0 0 0" />
+    <origin xyz="-0.039 0 0.0859" rpy="0 0 0"/>
+    <parent link="base_link"/>
+    <child link="odom_ground_truth"/>
   </joint>
   <!-- Camera -->
@@ -530,4 +568,15 @@
       <velocityGaussianNoise>0.005 0.005 0.05</velocityGaussianNoise>
     </plugin>
+    <plugin name="p3d_base_controller" filename="libgazebo_ros_p3d.so">
+      <alwaysOn>true</alwaysOn>
+      <updateRate>200.0</updateRate>
+      <bodyName>odom_ground_truth</bodyName>
+      <topicName>ground_truth/state_raw</topicName>
+      <gaussianNoise>0.00</gaussianNoise>
+      <frameName>world</frameName>
+      <!-- origin is at spawn location -->
+      <xyzOffset>0 8.5 0</xyzOffset>
+      <rpyOffset>0 0 0</rpyOffset>
+    </plugin>
     <!--<plugin name="tire_friction" filename="libTireFrictionPlugin.so">
       <link_name>left_rear_wheel</link_name>

Commit message: organized the gazebo files, and added first pass at CCRF track

File: autorally_description/urdf/autoRallyPlatform.urdf.xacro (robot description, xacro)
@@ -285,5 +285,5 @@
                  wheel_mass="${wheel_mass}"
                  axle_eff_limit="${axle_eff_limit}"
-                 wheel_model="package://autorally_description/urdf/autoRallyPlatformFrontWheelTextured.dae"
+                 wheel_model="package://autorally_description/urdf/cad/autoRallyPlatformFrontWheelTextured.dae"
                  cant="0.05"/>
   </xacro:macro>
@@ -299,5 +299,5 @@
                  wheel_mass="${wheel_mass}"
                  axle_eff_limit="${axle_eff_limit}"
-                 wheel_model="package://autorally_description/urdf/autoRallyPlatformRearWheelTextured.dae"
+                 wheel_model="package://autorally_description/urdf/cad/autoRallyPlatformRearWheelTextured.dae"
                  cant="-0.03"/>
   </xacro:macro>
@@ -321,5 +321,5 @@
               rpy="0 0 0"/>
       <geometry>
-        <mesh filename="package://autorally_description/urdf/Vehicle_Texture.dae" scale="1 1 1" />
+        <mesh filename="package://autorally_description/urdf/cad/Vehicle_Texture.dae" scale="1 1 1" />
       </geometry>
     </visual>
@@ -328,5 +328,5 @@
               rpy="0 0 0"/>
       <geometry>
-        <mesh filename="package://autorally_description/urdf/Vehicle_Texture.dae" scale="1 1 1" />
+        <mesh filename="package://autorally_description/urdf/cad/Vehicle_Texture.dae" scale="1 1 1" />
       </geometry>
     </collision>

Commit message: Merged everything but the controller with fork

File: autorally_description/urdf/autoRallyPlatform.urdf.xacro (robot description, xacro)
@@ -317,4 +317,9 @@
     <material>Gazebo/Grey</material>
   </gazebo>
+  <!-- Velodyne LIDAR -->
+  <xacro:include filename="$(find velodyne_description)/urdf/VLP-16.urdf.xacro"/>
+  <VLP-16 parent="base_link" name="velodyne" topic="/velodyne_points" hz="10" samples="440">
+    <origin xyz="0 0 ${chassis_height/2 + 0.075}" rpy="0 0 0" />
+  </VLP-16>
   <!-- Chassis -->
   <link name="chassis">
@@ -450,4 +455,12 @@
       <inertia ixx="1e-6" ixy="0" ixz="0" iyy="1e-6" iyz="0" izz="1e-6" />
     </inertial>
+  </link>
+  <!-- Reference frame for left camera (for stereo camera)-->
+  <joint name="left_camera_optical_joint" type="fixed">
+    <origin xyz="0 0.07 0" rpy="0 0 0"/>
+    <parent link="camera_link"/>
+    <child link="left_camera_optical_frame"/>
+  </joint>
+  <link name="left_camera_optical_frame">
   </link>
   <!-- camera -->

Commit message: Removed LIDAR components

File: autorally_description/urdf/autoRallyPlatform.urdf.xacro (robot description, xacro)
@@ -317,9 +317,4 @@
     <material>Gazebo/Grey</material>
   </gazebo>
-  <!-- Velodyne LIDAR -->
-  <xacro:include filename="$(find velodyne_description)/urdf/VLP-16.urdf.xacro"/>
-  <VLP-16 parent="base_link" name="velodyne" topic="/velodyne_points" hz="10" samples="440">
-    <origin xyz="0 0 ${chassis_height/2 + 0.075}" rpy="0 0 0" />
-  </VLP-16>
   <!-- Chassis -->
   <link name="chassis">
@@ -455,12 +450,4 @@
       <inertia ixx="1e-6" ixy="0" ixz="0" iyy="1e-6" iyz="0" izz="1e-6" />
     </inertial>
-  </link>
-  <!-- Reference frame for left camera (for stereo camera)-->
-  <joint name="left_camera_optical_joint" type="fixed">
-    <origin xyz="0 0.07 0" rpy="0 0 0"/>
-    <parent link="camera_link"/>
-    <child link="left_camera_optical_frame"/>
-  </joint>
-  <link name="left_camera_optical_frame">
   </link>
   <!-- camera -->
